File: Voyager50.kicad_pcb (KiCad board)
At the start: 2 copper layers, 244.5 x 76.2 mm, 192 parts, among them Q1 2N7002, SW1 5.2x5.2mm, U1 ATmega32U2-AU, U2 PRTR5V0U2X, Y1 16Mhz

Commit message: Finish routing
Parts:
- removed C1, C10, C11, C12, C13, C14, C15, C16, C17, C18, C5, C9: 0.1uF, Capacitors_SMD:C_0603
- removed D58, D62: SOD-123, Diodes_SMD:D_SOD-123
- removed G***: LOGO, locallib:ai-ring-6mm
- removed G***: LOGO, locallib:ai-4.8-ring
- removed K_ENTER3: MX-ISO, MX_Alps_Hybrid:MX-ISO-ReversedStabilizers
- removed K_LSPACE1: MX-2.25U, MX_Alps_Hybrid:MX-2.25U-ReversedStabilizers
- removed K_LSPACE2: MX-2.75U, MX_Alps_Hybrid:MX-2.75U-FLIPPED-ReversedStabilizers
- removed the K_RALT1 at (226.2, 96.8)
- removed K_RSHIFT2: MX-1.75U, MX_Alps_Hybrid:MX-1.75U
- removed K_RSHIFT3, K_SPACE3: MX-1U, MX_Alps_Hybrid:MX-1U
- removed K_RSHIFT4: MX-2.75U, MX_Alps_Hybrid:MX-2.75U
- removed K_RSPACE1: MX-2.75U, MX_Alps_Hybrid:MX-2.75U-ReversedStabilizers
- removed K_RSPACE2: MX-2.25U, MX_Alps_Hybrid:MX-2.25U-FLIPPED-ReversedStabilizers
- removed K_SPACE4: MX-1U, MX_Alps_Hybrid:MX-1U-FLIPPED
- removed R58, R62: 1k, Resistors_SMD:R_0805
- added D2: SOD-123, Diodes_SMD:D_SOD-123, B.Cu at (274.6, 57.1)
- added D3: SOD-123, Diodes_SMD:D_SOD-123, B.Cu at (265.1, 76.2)
- added D4: SOD-123, Diodes_SMD:D_SOD-123, B.Cu at (267.5, 95.2)
- added D5: SOD-123, Diodes_SMD:D_SOD-123, B.Cu at (288.9, 38.1)
- added D6: SOD-123, Diodes_SMD:D_SOD-123, B.Cu at (275.4, 76.2)
- added D7: SOD-123, Diodes_SMD:D_SOD-123, B.Cu at (291.3, 95.2)
- added K_'1: MX-1U, MX_Alps_Hybrid:MX-1U, F.Cu at (266.7, 58.7)
- added K_/1: MX-1U, MX_Alps_Hybrid:MX-1U, F.Cu at (257.2, 77.8)
- added K_ALT2: MX-1.5U, MX_Alps_Hybrid:MX-1.5U-FLIPPED, F.Cu at (95.2, 96.8)
- added K_CTRL2: MX-1.5U, MX_Alps_Hybrid:MX-1.5U-FLIPPED, F.Cu at (47.6, 96.8)
- added K_RALT2: MX-1.5U, MX_Alps_Hybrid:MX-1.5U, F.Cu at (257.2, 96.8)
- added K_RCTRL2: MX-1.5U, MX_Alps_Hybrid:MX-1.5U, F.Cu at (304.8, 96.8)
- added K_RMENU1: MX-1.25U, MX_Alps_Hybrid:MX-1.25U-FLIPPED, F.Cu at (283.4, 96.8)
- added K_RSHIFT1: MX-2.75U, MX_Alps_Hybrid:MX-2.75U, F.Cu at (292.9, 77.8)
- added K_RWIN1: MX-1.25U, MX_Alps_Hybrid:MX-1.25U-FLIPPED, F.Cu at (259.6, 96.8)
- added K_RWIN2: MX-1U, MX_Alps_Hybrid:MX-1U, F.Cu at (281.0, 96.8)
- added K_SPACE2: MX-7U, MX_Alps_Hybrid:MX-7U-ReversedStabilizers, F.Cu at (176.2, 96.8)
- added K_SRSHIFT1: MX-1.75U, MX_Alps_Hybrid:MX-1.75U, F.Cu at (283.4, 77.8)
- added K_WIN2: MX-1U, MX_Alps_Hybrid:MX-1U-FLIPPED, F.Cu at (71.4, 96.8)
- added K_[1: MX-1U, MX_Alps_Hybrid:MX-1U, F.Cu at (261.9, 39.7)
- added K_\2: MX-1U, MX_Alps_Hybrid:MX-1U, F.Cu at (285.8, 58.7)
- added K_]1: MX-1U, MX_Alps_Hybrid:MX-1U, F.Cu at (281.0, 39.7)
- added R2: 1k, Resistors_SMD:R_0603, B.Cu at (274.6, 62.7)
- added R3: 1k, Resistors_SMD:R_0603, B.Cu at (265.1, 81.8)
- added R4: 1k, Resistors_SMD:R_0603, B.Cu at (267.5, 100.8)
- added R5: 1k, Resistors_SMD:R_0603, B.Cu at (288.9, 43.7)
- added R6: 1k, Resistors_SMD:R_0603, B.Cu at (275.4, 81.8)
- added R7: 1k, Resistors_SMD:R_0603, B.Cu at (291.3, 100.8)
- added RGB13: WS2812B, LEDs:LED_WS2812B-PLCC4, B.Cu at (295.3, 49.2)
- added RGB14: WS2812B, LEDs:LED_WS2812B-PLCC4, B.Cu at (49.2, 87.3)
- K_ENTER2: value MX-1.25U -> MX-2.25U; footprint MX_Alps_Hybrid:MX-1.25U -> MX_Alps_Hybrid:MX-ISO-ReversedStabilizers
- K_RALT1: renamed from K_RWIN1; footprint MX_Alps_Hybrid:MX-1U -> MX_Alps_Hybrid:MX-1.25U
- K_RCTRL1: footprint MX_Alps_Hybrid:MX-1.25U -> MX_Alps_Hybrid:MX-1.25U-FLIPPED
- K_SPACE1: renamed from K_SPACE2; value MX-6U -> MX-6.25U; footprint MX_Alps_Hybrid:MX-6U-ReversedStabilizers -> MX_Alps_Hybrid:MX-6.25U-ReversedStabilizers
- K_SRSHIFT2: renamed from K_RSHIFT1; value MX-1.75U -> MX-1U; footprint MX_Alps_Hybrid:MX-1.75U -> MX_Alps_Hybrid:MX-1U
- K_WIN1: value MX-1U -> MX-1.25U; footprint MX_Alps_Hybrid:MX-1U -> MX_Alps_Hybrid:MX-1.25U
- R1, R16, R17, R18, R19, R20, R21, R22, R23, R24, R25, R26, R27, R31, R32, R33, R34, R35, R36, R37, R38, R39, R40, R41, R42, R44, R45, R46, R47, R48, R49, R50, R51, R52, R53, R54, R55, R59, R60, R61, R63, R64, R67, R68, R70, R71, R72, R73, R74: footprint Resistors_SMD:R_0805 -> Resistors_SMD:R_0603
- R69: value 1k -> 100; footprint Resistors_SMD:R_0805 -> Resistors_SMD:R_0603
- SW1: value 5.2x5.2mm -> SW_Push
- U1: value ATmega32U2-AU -> ATmega32U2-MU
- moved D55 74.6 mm to (301.6, 76.2)
- moved R55 74.6 mm to (301.6, 81.8)
- moved D1 68.7 mm to (269.9, 38.1)
- moved R1 68.7 mm to (269.9, 43.7)
- moved RGB6 50.8 mm to (220.7, 87.3)
- moved RGB8 49.2 mm to (176.2, 87.3)
- moved RGB4 46.8 mm to (261.9, 87.3)
- moved RGB10 45.2 mm to (133.3, 87.3)
- moved K_SRSHIFT2 45.2 mm to (309.6, 77.8)
- moved D42 41.3 mm to (277.8, 57.1)
- moved R42 41.3 mm to (277.8, 62.7)
- moved RGB12 41.3 mm to (90.5, 87.3)
- moved K_ENTER2 39.3 mm to (307.2, 49.2)
- moved D27 38.1 mm to (292.1, 38.1)
- moved K_ENTER1 38.1 mm to (297.7, 58.7)
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Connections:
- net .-COL renamed COL10
- net .-LEDGND renamed Net-(K_.1-Pad4)
- net .-ROW renamed Net-(D54-Pad2)
- D1 pad 1: ROW3 -> ROW0
- K_ENTER1 pad 1: COL11 -> COL13
- K_ENTER2 pad 1: Net-(D42-Pad2) -> COL13
- K_ENTER2 pad 2: COL11 -> Net-(D42-Pad2)
- K_RCTRL1 pad 1: COL11 -> COL13
- K_SRSHIFT2 pad 1: COL11 -> COL13
- K_\1 pad 1: COL11 -> COL13
- RGB2 pad 4: Net-(RGB11-Pad2) -> Net-(RGB13-Pad2)
- U1 pad 10: ROW2 -> ROW3
- U1 pad 11: ROW3 -> COL13
- U1 pad 12: COL11 -> COL12
- U1 pad 13: Net-(R71-Pad2) -> COL11
- U1 pad 25: ROW1 -> COL1
- U1 pad 26: RGBLED -> COL0
- U1 pad 33: (no net) -> GND
- U1 pad 5: Net-(U1-Pad5) -> RGBLED
- U1 pad 6: Net-(U1-Pad6) -> ROW0
- U1 pad 7: COL0 -> Net-(R71-Pad2)
- U1 pad 8: COL1 -> ROW1
- U1 pad 9: ROW0 -> ROW2
Routing:
- net COL13: track 0.00 -> 352.0 mm, vias 0 -> 1
- net COL12: track 0.00 -> 294.7 mm
- net LEDGND: track 871.0 -> 998.8 mm
- net +5V: track 1290.8 -> 1382.8 mm
- net ROW2: track 220.7 -> 299.1 mm
- net GND: track 652.9 -> 729.8 mm, vias 21 -> 6
- net COL11: track 318.8 -> 258.7 mm, vias 1 -> 0
- net ROW0: track 244.2 -> 299.5 mm, vias 4 -> 3
- net Net-(RGB13-Pad2): track 0.00 -> 50.9 mm, vias 0 -> 2
- net ROW1: track 220.5 -> 270.2 mm
- net Net-(K_SRSHIFT2-Pad4): track 52.4 -> 10.4 mm
- net Net-(RGB12-Pad2): track 0.00 -> 39.8 mm
- net COL4: track 136.0 -> 105.3 mm
- net COL8: track 209.6 -> 178.9 mm
- net Net-(D6-Pad2): track 0.00 -> 28.9 mm
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Other:
- board size 244.5 x 76.2 mm -> 282.6 x 76.2 mm
- board text removed: "40"
- board text removed: "VOYAGER"
- board text removed: "Voyager40 PCB Rev 1.0 20190203"
- board text removed: "kb.ai03.me"
