File: Voyager50.sch (KiCad schematic (older format))
At the start: 190 parts, among them Q1 2N7002, SW1 5.2x5.2mm, U1 ATmega32U2-AU, U2 PRTR5V0U2X, Y1 16Mhz

Commit message: Finish routing
Parts:
- removed C1, C10, C11, C12, C13, C14, C15, C16, C17, C18, C5, C9: 0.1uF, Capacitors_SMD:C_0603, symbol Device:C_Small
- removed D58, D62: SOD-123, Diodes_SMD:D_SOD-123, symbol Device:D_Small
- removed K_ENTER3: MX-ISO, MX_Alps_Hybrid:MX-ISO-ReversedStabilizers, symbol MX_Alps_Hybrids:MX-1U
- removed K_LSPACE1: MX-2.25U, MX_Alps_Hybrid:MX-2.25U-ReversedStabilizers, symbol MX_Alps_Hybrids:MX-1U
- removed K_LSPACE2: MX-2.75U, MX_Alps_Hybrid:MX-2.75U-FLIPPED-ReversedStabilizers, symbol MX_Alps_Hybrids:MX-1U
- removed K_RALT1: MX-1.25U, MX_Alps_Hybrid:MX-1.25U, symbol MX_Alps_Hybrids:MX-1U
- removed K_RSHIFT2: MX-1.75U, MX_Alps_Hybrid:MX-1.75U, symbol MX_Alps_Hybrids:MX-1U
- removed K_RSHIFT3, K_SPACE3: MX-1U, MX_Alps_Hybrid:MX-1U, symbol MX_Alps_Hybrids:MX-1U
- removed K_RSHIFT4: MX-2.75U, MX_Alps_Hybrid:MX-2.75U, symbol MX_Alps_Hybrids:MX-1U
- removed K_RSPACE1: MX-2.75U, MX_Alps_Hybrid:MX-2.75U-ReversedStabilizers, symbol MX_Alps_Hybrids:MX-1U
- removed K_RSPACE2: MX-2.25U, MX_Alps_Hybrid:MX-2.25U-FLIPPED-ReversedStabilizers, symbol MX_Alps_Hybrids:MX-1U
- removed K_SPACE4: MX-1U, MX_Alps_Hybrid:MX-1U-FLIPPED, symbol MX_Alps_Hybrids:MX-1U
- removed R58, R62: 1k, Resistors_SMD:R_0805, symbol Device:R_Small
- removed SW1: 5.2x5.2mm, random-keyboard-parts:SKQGADE010, symbol Voyager40-rescue:SW_Push-Voyager60-rescue
- removed U1: ATmega32U2-AU, Housings_DFN_QFN:QFN-32-1EP_5x5mm_Pitch0.5mm, symbol Voyager40-rescue:ATmega32U2-AU-MCU_Microchip_ATmega
- added D2, D3, D4, D5, D6, D7: SOD-123, Diodes_SMD:D_SOD-123, symbol Device:D_Small
- added K_'1, K_/1, K_RWIN2, K_[1, K_\2, K_]1: MX-1U, MX_Alps_Hybrid:MX-1U, symbol MX_Alps_Hybrids:MX-1U
- added K_ALT2, K_CTRL2: MX-1.5U, MX_Alps_Hybrid:MX-1.5U-FLIPPED, symbol MX_Alps_Hybrids:MX-1U
- added K_RALT2, K_RCTRL2: MX-1.5U, MX_Alps_Hybrid:MX-1.5U, symbol MX_Alps_Hybrids:MX-1U
- added K_RMENU1, K_RWIN1: MX-1.25U, MX_Alps_Hybrid:MX-1.25U-FLIPPED, symbol MX_Alps_Hybrids:MX-1U
- added K_RSHIFT1: MX-2.75U, MX_Alps_Hybrid:MX-2.75U, symbol MX_Alps_Hybrids:MX-1U
- added K_SPACE2: MX-7U, MX_Alps_Hybrid:MX-7U-ReversedStabilizers, symbol MX_Alps_Hybrids:MX-1U
- added K_SRSHIFT1: MX-1.75U, MX_Alps_Hybrid:MX-1.75U, symbol MX_Alps_Hybrids:MX-1U
- added K_WIN2: MX-1U, MX_Alps_Hybrid:MX-1U-FLIPPED, symbol MX_Alps_Hybrids:MX-1U
- added R2, R3, R4, R5, R6, R7: 1k, Resistors_SMD:R_0603, symbol Device:R_Small
- added RGB13, RGB14: WS2812B, LEDs:LED_WS2812B-PLCC4, symbol LED:WS2812B
- added SW1: SW_Push, random-keyboard-parts:SKQGADE010, symbol Switch:SW_Push
- added U1: ATmega32U2-MU, Housings_DFN_QFN:QFN-32-1EP_5x5mm_Pitch0.5mm, symbol MCU_Microchip_ATmega:ATmega32U2-MU
- K_ENTER2: value MX-1.25U -> MX-2.25U; footprint MX_Alps_Hybrid:MX-1.25U -> MX_Alps_Hybrid:MX-ISO-ReversedStabilizers
- K_RALT1: renamed from K_RWIN1; footprint MX_Alps_Hybrid:MX-1U -> MX_Alps_Hybrid:MX-1.25U
- K_RCTRL1: footprint MX_Alps_Hybrid:MX-1.25U -> MX_Alps_Hybrid:MX-1.25U-FLIPPED
- K_SPACE1: renamed from K_SPACE2; value MX-6U -> MX-6.25U; footprint MX_Alps_Hybrid:MX-6U-ReversedStabilizers -> MX_Alps_Hybrid:MX-6.25U-ReversedStabilizers
- K_SRSHIFT2: renamed from K_RSHIFT1; value MX-1.75U -> MX-1U; footprint MX_Alps_Hybrid:MX-1.75U -> MX_Alps_Hybrid:MX-1U
- K_WIN1: value MX-1U -> MX-1.25U; footprint MX_Alps_Hybrid:MX-1U -> MX_Alps_Hybrid:MX-1.25U
- R1, R16, R17, R18, R19, R20, R21, R22, R23, R24, R25, R26, R27, R31, R32, R33, R34, R35, R36, R37, R38, R39, R40, R41, R42, R44, R45, R46, R47, R48, R49, R50, R51, R52, R53, R54, R55, R59, R60, R61, R63, R64, R67, R68, R70, R71, R72, R73, R74: footprint Resistors_SMD:R_0805 -> Resistors_SMD:R_0603
- R69: value 1k -> 100; footprint Resistors_SMD:R_0805 -> Resistors_SMD:R_0603
Connections:
- net labels added: COL12, COL13
- net labels removed: .-COL, .-LEDGND, .-ROW
- wire segments 533 -> 535
Other:
- moved on the sheet: C6, D27, D42, D55, D64, K_ENTER1, K_RCTRL1, K_SRSHIFT2, K_\1, R27, R42, R55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
